File: KiCAD/line_follower_design_4/line_follower_design_4_Mk_II.kicad_pcb (KiCad board)
At the start: 2 copper layers, 101.6 x 99.1 mm, 50 parts, among them M1 Motor Levi, M2 Motor Desni, Q1 Q_NPN_BCE, Q2 BSS138, Q3 BSS138, Q4 Q_PMOS_GDS, SW1 switch_psh, SW2 switch, U1 MCP1703A-5002/MB

Commit message: line-follower-design-4 schematic update, pcb update
Library dependencies update, PCB components optimizations.
Parts:
- Q1: footprint BCE547B(T0-92):BCE547B(T0-92) -> Transistors_OldSowjetAera:OldSowjetaera_Transistor_Type-I_SmallPads
- moved Q1 2.27 mm to (-27.9, 121.9)
Other:
- board outline removed
Changed lines of the file:
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@@
     (links 132)
     (no_connects 132)
-    (area -122.020001 53.239999 -20.219999 152.500001)
+    (area -122.37 50.35 -13.469999 152.500001)
     (thickness 1.6)
     (drawings 5)
@@
     (trace_min 0.2)
     (segment_width 0.2)
-    (edge_width 0.2)
+    (edge_width 0.15)
     (via_size 0.6)
     (via_drill 0.4)
@@
     (pad_to_mask_clearance 0.2)
     (aux_axis_origin 0 0)
-    (visible_elements 7FFFF7FF)
+    (visible_elements 7FFFFFFF)
     (pcbplotparams
       (layerselection 0x00030_80000001)
@@
       (net 3 GND))
   )
+  (module Transistors_OldSowjetAera:OldSowjetaera_Transistor_Type-I_SmallPads (layer F.Cu)
+    (at -27.94 121.92)
+    (fp_text reference Q1 (at 0 -7.1) (layer F.SilkS)
+      (effects (font (size 1 1) (thickness 0.15)))
+    )
+    (fp_text value Q_NPN_BCE (at 0.1 7.6) (layer F.Fab)
+      (effects (font (size 1 1) (thickness 0.15)))
+    )
+    (fp_circle (center -4.8 0) (end -4.8 0.4) (layer F.SilkS) (width 0.15))
+    (fp_circle (center 0 0) (end 4 0) (layer F.SilkS) (width 0.15))
+    (fp_circle (center 0 0) (end 5.6 0) (layer F.SilkS) (width 0.15))
+    (pad 2 thru_hole circle (at 0 0) (size 1.4 1.4) (drill 0.8) (layers *.Cu *.Mask)
+      (net 48 "Net-(Q1-Pad2)"))
+    (pad 1 thru_hole circle (at -2 0) (size 1.4 1.4) (drill 0.8) (layers *.Cu *.Mask)
+      (net 49 "Net-(Q1-Pad1)"))
+    (pad 3 thru_hole circle (at 2 0) (size 1.4 1.4) (drill 0.8) (layers *.Cu *.Mask)
+      (net 3 GND))
+    (model Transistors_OldSowjetAera.3dshapes/OldSowjetaera_Transistor_Type-I_SmallPads.wrl
+      (at (xyz 0 0 0))
+      (scale (xyz 0.3937 0.3937 0.3937))
+      (rotate (xyz 0 0 0))
+    )
+  )
   (module TO_SOT_Packages_SMD:SOT-23 (layer F.Cu)
     (at -43.18 101.6 270)
@@
       (net 18 "Net-(BT1-Pad31)"))
   )
-  (module "BCE547B(T0-92):BCE547B(T0-92)" (layer F.Cu)
-    (at -28.956 119.888)
-    (fp_text reference Q1 (at 2.54 0.508) (layer F.SilkS)
-      (effects (font (size 1 1) (thickness 0.15)))
-    )
-    (fp_text value Q_NPN_BCE (at 2.286 -5.588) (layer F.Fab)
-      (effects (font (size 1 1) (thickness 0.15)))
-    )
-    (fp_line (start 5.334 -3.81) (end 5.334 -4.318) (layer F.SilkS) (width 0.15))
-    (fp_line (start -0.762 -3.81) (end -0.762 -4.318) (layer F.SilkS) (width 0.15))
-    (fp_line (start -0.762 -4.318) (end 5.334 -4.318) (layer F.SilkS) (width 0.15))
-    (fp_arc (start 2.286 -3.81) (end 2.286 -0.762) (angle 90) (layer F.SilkS) (width 0.15))
-    (fp_arc (start 2.286 -3.81) (end 5.334 -3.81) (angle 90) (layer F.SilkS) (width 0.15))
-    (pad 1 thru_hole circle (at 3.556 -3.302) (size 1 1) (drill 0.7) (layers *.Cu *.Mask)
-      (net 49 "Net-(Q1-Pad1)"))
-    (pad 2 thru_hole circle (at 2.286 -3.302) (size 1 1) (drill 0.7) (layers *.Cu *.Mask)
-      (net 48 "Net-(Q1-Pad2)"))
-    (pad 3 thru_hole circle (at 1.016 -3.302) (size 1 1) (drill 0.7) (layers *.Cu *.Mask)
-      (net 3 GND))
-  )
-  (gr_line (start -20.32 53.848) (end -20.32 53.34) (angle 90) (layer Edge.Cuts) (width 0.2))
-  (gr_line (start -20.32 152.4) (end -20.32 53.848) (angle 90) (layer Edge.Cuts) (width 0.2))
-  (gr_line (start -121.92 152.4) (end -20.32 152.4) (angle 90) (layer Edge.Cuts) (width 0.2))
-  (gr_line (start -121.92 53.34) (end -121.92 152.4) (angle 90) (layer Edge.Cuts) (width 0.2))
-  (gr_line (start -20.32 53.34) (end -121.92 53.34) (angle 90) (layer Edge.Cuts) (width 0.2))
+  (gr_line (start -20.32 53.848) (end -20.32 53.34) (angle 90) (layer B.Adhes) (width 0.2))
+  (gr_line (start -20.32 152.4) (end -20.32 53.848) (angle 90) (layer B.Adhes) (width 0.2))
+  (gr_line (start -121.92 152.4) (end -20.32 152.4) (angle 90) (layer B.Adhes) (width 0.2))
+  (gr_line (start -121.92 53.34) (end -121.92 152.4) (angle 90) (layer B.Adhes) (width 0.2))
+  (gr_line (start -20.32 53.34) (end -121.92 53.34) (angle 90) (layer B.Adhes) (width 0.2))
   (zone (net 0) (net_name "") (layer F.Cu) (hatch edge 0.508)
     (connect_pads (clearance 0.508))
